File: mp3_clean/mp3/mp3.kicad_sch (KiCad schematic)
At the start: 57 parts, among them J1 USB4105-GF-A, J2 LEFT, J3 DEBUG, J4 RIGHT, Q1 FDG6320C, SW1 PCM12, U1 W25Q128JV, U2 RP2040, U3 MCP1702T-3302E_CB, U4 MCP73831T-2ACI_OT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

Commit message: update
Connections:
- net GPIO26 is gone; now on net GND: J4.10 (Pin_10), U2.38 (GPIO26/ADC0)
- net GPIO19: now also Q1.2, R14.1
Changed lines of the file:
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@@
   (junction (at 24.13 120.65) (diameter 0) (color 0 0 0 0)
   )
+  (junction (at 212.09 68.58) (diameter 0) (color 0 0 0 0)
+  )
   (junction (at 43.18 81.28) (diameter 0) (color 0 0 0 0)
+  )
+  (junction (at 241.3 86.36) (diameter 0) (color 0 0 0 0)
   )
   (junction (at 252.73 67.31) (diameter 0) (color 0 0 0 0)
@@
     (stroke (width 0) (type default) (color 0 0 0 0))
   )
+  (wire (pts (xy 231.14 86.36) (xy 241.3 86.36))
+    (stroke (width 0) (type default) (color 0 0 0 0))
+  )
   (wire (pts (xy 80.01 186.69) (xy 80.01 191.77))
     (stroke (width 0) (type default) (color 0 0 0 0))
@@
     (stroke (width 0) (type default) (color 0 0 0 0))
   )
+  (wire (pts (xy 196.85 68.58) (xy 212.09 68.58))
+    (stroke (width 0) (type default) (color 0 0 0 0))
+  )
   (wire (pts (xy 356.87 24.13) (xy 356.87 26.67))
     (stroke (width 0) (type default) (color 0 0 0 0))
@@
     (effects (font (size 1.27 1.27)) (justify right bottom))
   )
+  (label "GPIO26" (at 196.85 68.58 0)
+    (effects (font (size 1.27 1.27)) (justify left bottom))
+  )
   (label "GPIO17" (at 200.66 161.29 180)
     (effects (font (size 1.27 1.27)) (justify right bottom))
@@
     (effects (font (size 1.27 1.27)) (justify left bottom))
   )
+  (label "GPIO19" (at 231.14 86.36 0)
+    (effects (font (size 1.27 1.27)) (justify left bottom))
+  )
