File: mp3_complete/mp3/mp3.kicad_sch (KiCad schematic)
At the start: 57 parts, among them J1 USB4105-GF-A, J2 LEFT, J3 DEBUG, J4 RIGHT, Q1 FDG6320C, SW1 PCM12, U1 W25Q128JV, U2 RP2040, U3 MCP1702T-3302E_CB, U4 MCP73831T-2ACI_OT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

Commit message: finished mp3_complete
Parts:
- added SW2: SW_MEC_5G, symbol Switch:SW_MEC_5G
Connections:
- net +3V3: now also SW2.3 (B), SW2.4 (B)
- net GPIO20: now also SW2.1 (A), SW2.2 (A)
- net GPIO21: now also J_st7735r.11 (Pin_11)
- net GPIO22: now also J_st7735r.12 (Pin_12)
- net GPIO23: now also J_st7735r.13 (Pin_13)
- net GPIO24: now also J_st7735r.14 (Pin_14)
Other:
- moved on the sheet: J2, J3, J4
