File: PicoCam_DowlingZachary/PicoCam_DowlingZachary/PicoCam_DowlingZachary.kicad_pcb (KiCad board)
At the start: 2 copper layers, 50.8 x 44.5 mm, 56 parts, among them J1 USB4105-GF-A, J2 S2B-PH-SM4-TB, J3 DEBUG, Q1 FDG6320C, SW1 PCM12, U1 W25Q128JV, U2 RP2040, U3 MCP1702T-3302E_CB, U4 MCP73831T-2ACI_OT, U5 TPS2113APW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

Commit message: update
Parts:
- removed OlinLogoLg1: G***, Eclectronics:OlinLogoLg1
Other:
- board text removed: "0 1 G 2 3 4 5 G 6 7 8 9 G 10 11 12 13 G 14 15"
- board text removed: "B 23 G BOOT 3V3 29 28 G 27 26 RUN 22 G 21 20 19 18 G 17 16"
- board text removed: "BOOT"
- board text removed: "DEBUG"
- board text removed: "PWR"
- board text removed: "RESET"
- board text removed: "SWCLK GND SWDIO"
- board text removed: "Zachary Sherman 2022"
- board text removed: "Zachberry Pi Pico V1"
Changed lines of the file:
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@@
     (pad "S2" smd rect locked (at 3.35 -5.75) (size 1.5 3.4) (layers "B.Cu" "B.Paste" "B.Mask"))
-  )
-  (footprint "Eclectronics:OlinLogoLg1" (layer "B.Cu")
-    (at 104.82 44.73 180)
-    (descr "Imported from OlinLogo.svg")
-    (tags "svg2mod")
-    (attr smd)
-    (fp_text reference "OlinLogoLg1" (at 0 5.204532) (layer "B.SilkS") hide
-      (effects (font (size 1.524 1.524) (thickness 0.3048)) (justify mirror))
-    )
-    (fp_text value "G***" (at 0 -5.204532) (layer "B.SilkS") hide
-      (effects (font (size 1.524 1.524) (thickness 0.3048)) (justify mirror))
-    )
-    (fp_poly (pts
-        (xy 1.736725 1.923058)
-        (xy 1.869952 1.730127)
-        (xy 1.922487 1.466001)
-        (xy 1.894562 1.14116)
-        (xy 1.786406 0.766086)
-        (xy 1.598251 0.351262)
-        (xy 1.330327 -0.092831)
-        (xy 1.075434 -0.440325)
-        (xy 0.797385 -0.766282)
-        (xy 0.502598 -1.066073)
-        (xy 0.197493 -1.335068)
-        (xy -0.111511 -1.568637)
-        (xy -0.417994 -1.762151)
-        (xy -0.715537 -1.910981)
-        (xy -0.997721 -2.010496)
-        (xy -0.560127 -2.030364)
-        (xy -0.122631 -2.027922)
-        (xy 0.311568 -2.003984)
-        (xy 0.739273 -1.959364)
-        (xy 1.157284 -1.894876)
-        (xy 1.562404 -1.811334)
-        (xy 1.951435 -1.70955)
-        (xy 2.321177 -1.59034)
-        (xy 2.668433 -1.454516)
-        (xy 2.990005 -1.302893)
-        (xy 3.282694 -1.136284)
-        (xy 3.543302 -0.955502)
-        (xy 3.768631 -0.761363)
-        (xy 3.955482 -0.554678)
-        (xy 4.122829 -0.292971)
-        (xy 4.217397 -0.032265)
-        (xy 4.241806 0.224727)
-        (xy 4.198677 0.475294)
-        (xy 4.090631 0.716723)
-        (xy 3.920287 0.946303)
-        (xy 3.690266 1.16132)
-        (xy 3.403189 1.359064)
-        (xy 3.061676 1.536822)
-        (xy 2.668347 1.691881)
-        (xy 2.225823 1.821531)
-        (xy 1.736725 1.923058)
-      ) (layer "B.SilkS") (width 0) (fill solid))
-    (fp_poly (pts
-        (xy 0.997721 2.010441)
-        (xy 0.560139 2.030319)
-        (xy 0.122654 2.027887)
-        (xy -0.311534 2.003957)
-        (xy -0.739228 1.959343)
-        (xy -1.15723 1.894859)
-        (xy -1.562342 1.811319)
-        (xy -1.951366 1.709537)
-        (xy -2.321103 1.590325)
-        (xy -2.668356 1.454499)
-        (xy -2.989927 1.302872)
-        (xy -3.282617 1.136256)
-        (xy -3.543229 0.955467)
-        (xy -3.768565 0.761318)
-        (xy -3.955426 0.554623)
-        (xy -4.122784 0.292916)
-        (xy -4.217357 0.03221)
-        (xy -4.241768 -0.224782)
-        (xy -4.198639 -0.475347)
-        (xy -4.09059 -0.716774)
-        (xy -3.920245 -0.946351)
-        (xy -3.690226 -1.161365)
-        (xy -3.403154 -1.359103)
-        (xy -3.061652 -1.536854)
-        (xy -2.66834 -1.691905)
-        (xy -2.225843 -1.821543)
-        (xy -1.736781 -1.923058)
-        (xy -1.869969 -1.730151)
-        (xy -1.922493 -1.46604)
-        (xy -1.894575 -1.141208)
-        (xy -1.786437 -0.76614)
-        (xy -1.598299 -0.351317)
-        (xy -1.330382 0.092776)
-        (xy -1.075485 0.440288)
-        (xy -0.797423 0.766258)
-        (xy -0.502621 1.066057)
-        (xy -0.197499 1.335054)
-        (xy 0.111518 1.568621)
-        (xy 0.418009 1.762127)
-        (xy 0.715551 1.910944)
-        (xy 0.997721 2.010441)
-      ) (layer "B.SilkS") (width 0) (fill solid))
   )
   (footprint "Connector_PinHeader_2.54mm:PinHeader_2x09_P2.54mm_Vertical" (layer "B.Cu")
@@
   (gr_line (start 97.538206 125.412183) (end 97.439493 125.429812) (layer "Edge.Cuts") (width 0.1))
   (gr_line (start 48.859486 81.65963) (end 48.925858 81.590014) (layer "Edge.Cuts") (width 0.1))
-  (gr_text "SWCLK\nGND\nSWDIO" (at 73.06 46.23) (layer "B.SilkS")
-    (effects (font (size 1.5748 1.5748) (thickness 0.15)) (justify right mirror))
-  )
-  (gr_text "B\n23\nG\nBOOT\n3V3\n29\n28\nG\n27\n26\nRUN\n22\nG\n21\n20\n19\n18\nG\n17\n16" (at 94.69 53.03 270) (layer "B.SilkS")
-    (effects (font (size 1.5748 1.5748) (thickness 0.15)) (justify left mirror))
-  )
-  (gr_text "0\n1\nG\n2\n3\n4\n5\nG\n6\n7\n8\n9\nG\n10\n11\n12\n13\nG\n14\n15" (at 94.79 39.07 270) (layer "B.SilkS")
-    (effects (font (size 1.5748 1.5748) (thickness 0.15)) (justify right mirror))
-  )
-  (gr_text "Zachary Sherman\n2022" (at 99.74 44.78) (layer "B.SilkS")
-    (effects (font (size 1.27 1.27) (thickness 0.15)) (justify left mirror))
-  )
-  (gr_text "Zachberry Pi Pico V1" (at 80.29 40.485) (layer "F.SilkS")
-    (effects (font (size 1.27 1.27) (thickness 0.15)))
-  )
-  (gr_text "DEBUG" (at 73.665 46.31 270) (layer "F.SilkS")
-    (effects (font (size 1 1) (thickness 0.15)))
-  )
-  (gr_text "PWR" (at 79.94 46.935 90) (layer "F.SilkS")
-    (effects (font (size 1 1) (thickness 0.15)))
-  )
-  (gr_text "RESET" (at 84.19 52.26) (layer "F.SilkS")
-    (effects (font (size 1 1) (thickness 0.15)))
-  )
-  (gr_text "BOOT\n" (at 113.99 52.41) (layer "F.SilkS")
-    (effects (font (size 1 1) (thickness 0.15)))
-  )
   (segment (start 58.965 113.01) (end 58.965 110.985) (width 0.1524) (layer "F.Cu") (net 1))
   (segment (start 76.6848 97.83) (end 76.68 97.8348) (width 0.1524) (layer "F.Cu") (net 1))
@@
     (connect_pads (clearance 0))
     (min_thickness 0.254)
-    (keepout (tracks allowed) (vias allowed) (pads allowed) (copperpour not_allowed) (footprints allowed))
+    (keepout (tracks allowed) (vias allowed) (pads allowed ) (copperpour not_allowed) (footprints allowed))
     (fill (thermal_gap 0.508) (thermal_bridge_width 0.508))
     (polygon
